Commit message: finished robot

File: colcon_ws/src/robot/urdf/robot.xacro (robot description, xacro)
@@ -6,4 +6,5 @@
   <xacro:include filename="$(find robot)/urdf/parts/right_thigh/right_thigh.xacro"/>
   <xacro:include filename="$(find robot)/urdf/parts/shin/shin.xacro"/>
+    <xacro:include filename="$(find robot)/urdf/robot_control_gazebo.xacro"/>
   <xacro:property name="PI" value="3.14159274"/>
   <!-- =============== Link & Joint =============== -->
@@ -64,4 +65,5 @@
   <!-- Controllers -->
   <!-- Base -->
+  <!-- Base -->
   <xacro:base_gazebo_v0/>
   <xacro:leg_joint_gazebo_v0 prefix="rear_left"/>

File: colcon_ws/src/robot/urdf/robot_control_gazebo.xacro (robot description, xacro)
@@ -1,79 +1,121 @@
-<?xml version="1.0"?>
-<robot name="acs_robot" xmlns:xacro="http://ros.org/wiki/xacro">
-  <xacro:include filename="$(find robot)/urdf/parts/base/base.xacro"/>
-  <xacro:include filename="$(find robot)/urdf/parts/leg_joint/leg_joint.xacro"/>
-  <xacro:include filename="$(find robot)/urdf/parts/left_thigh/left_thigh.xacro"/>
-  <xacro:include filename="$(find robot)/urdf/parts/right_thigh/right_thigh.xacro"/>
-  <xacro:include filename="$(find robot)/urdf/parts/shin/shin.xacro"/>
-  <xacro:property name="PI" value="3.14159274"/>
-  <!-- =============== Link & Joint =============== -->
-  <!-- Base -->
-  <!-- <link name="base_footprint"/> -->
-  <xacro:base parent="base_footprint">
-    <origin xyz="0 0 0" rpy="0 0 0" />
-  </xacro:base>
-  <xacro:leg_joint_v0 prefix="rear_left" parent="base_link">
-    <origin xyz="-0.277 0.06 0.089405" rpy="0 ${PI/2} ${-PI/2}"/>
-    <axis xyz="0 -1 0"/> <!-- 0 -1 0 -->
-  </xacro:leg_joint_v0>
-  <xacro:leg_joint_v0 prefix="rear_right" parent="base_link">
-    <origin xyz="-0.277 -0.06 0.089405" rpy="0 ${-PI/2} ${-PI/2}"/>
-    <axis xyz="0 1 0"/>
-  </xacro:leg_joint_v0>
-  <xacro:leg_joint_v0 prefix="front_left" parent="base_link">
-    <origin xyz="0.282 0.06 0.090255" rpy="0 ${PI/2} ${-PI/2}"/>
-    <axis xyz="0 -1 0"/> <!-- 0 -1 0 -->
-  </xacro:leg_joint_v0>
-  <xacro:leg_joint_v0 prefix="front_right" parent="base_link">
-    <origin xyz="0.282 -0.06 0.090255" rpy="0 ${-PI/2} ${-PI/2}"/>
-    <axis xyz="0 1 0"/>
-  </xacro:leg_joint_v0>
-  <xacro:left_thigh_v0 prefix="front" parent="front_left_leg_joint_link">
-    <origin xyz="0 0 -0.114" rpy="${PI/2} 0 ${-PI/2}"/>
-    <axis xyz="0 1 0"/>
-  </xacro:left_thigh_v0>
-  <xacro:left_thigh_v0 prefix="rear" parent="rear_left_leg_joint_link">
-    <origin xyz="0 0 -0.114" rpy="${PI/2} 0 ${-PI/2}"/>
-    <axis xyz="0 1 0"/>
-  </xacro:left_thigh_v0>
-  <xacro:right_thigh_v0 prefix="front" parent="front_right_leg_joint_link">
-    <origin xyz="0 0 -0.114" rpy="${PI/2} 0 ${-PI/2}"/>
-    <axis xyz="0 -1 0"/> <!-- 0 -1 0 -->
-  </xacro:right_thigh_v0>
-  <xacro:right_thigh_v0 prefix="rear" parent="rear_right_leg_joint_link">
-    <origin xyz="0 0 -0.114" rpy="${PI/2} 0 ${-PI/2}"/>
-    <axis xyz="0 -1 0"/> <!-- 0 -1 0 -->
-  </xacro:right_thigh_v0>
-  <xacro:shin_v0 prefix="front_left" parent="front_left_thigh_link">
-    <origin xyz="0.426 -0.0285 0" rpy="0 0 0"/>
-    <axis xyz="0 1 0"/>
-  </xacro:shin_v0>
-  <xacro:shin_v0 prefix="front_right" parent="front_right_thigh_link">
-    <origin xyz="0.426 -0.0285 0" rpy="${PI} 0 0"/>
-    <axis xyz="0 1 0"/>
-  </xacro:shin_v0>
-  <xacro:shin_v0 prefix="rear_left" parent="rear_left_thigh_link">
-    <origin xyz="0.426 -0.0285 0" rpy="0 0 0"/>
-    <axis xyz="0 1 0"/>
-  </xacro:shin_v0>
-  <xacro:shin_v0 prefix="rear_right" parent="rear_right_thigh_link">
-    <origin xyz="0.426 -0.0285 0" rpy="${PI} 0 0"/>
-    <axis xyz="0 1 0"/>
-  </xacro:shin_v0>
-  <!-- =============== Gazebo =============== -->
-  <!-- Controllers -->
-  <!-- Base -->
-  <xacro:base_gazebo_v0/>
-  <xacro:leg_joint_gazebo_v0 prefix="rear_left"/>
-  <xacro:leg_joint_gazebo_v0 prefix="front_left"/>
-  <xacro:leg_joint_gazebo_v0 prefix="rear_right"/>
-  <xacro:leg_joint_gazebo_v0 prefix="front_right"/>
-  <xacro:left_thigh_gazebo_v0 prefix="front"/>
-  <xacro:left_thigh_gazebo_v0 prefix="rear"/>
-  <xacro:right_thigh_gazebo_v0 prefix="front"/>
-  <xacro:right_thigh_gazebo_v0 prefix="rear"/>
-  <xacro:shin_gazebo_v0 prefix="rear_left"/>
-  <xacro:shin_gazebo_v0 prefix="front_left"/>
-  <xacro:shin_gazebo_v0 prefix="rear_right"/>
-  <xacro:shin_gazebo_v0 prefix="front_right"/>
+<?xml version="1.0" ?>
+<robot xmlns:xacro="http://www.ros.org/wiki/xacro">
+<xacro:macro name="robot_ros2_control">
+    <ros2_control name="fws" type="system">
+      <hardware>
+          <plugin>gz_ros2_control/GazeboSimSystem</plugin>
+      </hardware>
+    <joint name="front_left_leg_joint">
+      <command_interface name="position">
+        <param name="min">-3.14</param>
+        <param name="max">3.14</param>
+      </command_interface>
+      <state_interface name="position"/>
+    </joint>
+    <joint name="front_right_leg_joint">
+      <command_interface name="position">
+        <param name="min">-3.14</param>
+        <param name="max">3.14</param>
+      </command_interface>
+      <state_interface name="position"/>
+    </joint>
+    <joint name="rear_left_leg_joint">
+      <command_interface name="position">
+        <param name="min">-3.14</param>
+        <param name="max">3.14</param>
+      </command_interface>
+      <state_interface name="position"/>
+    </joint>
+    <joint name="rear_right_leg_joint">
+      <command_interface name="position">
+        <param name="min">-3.14</param>
+        <param name="max">3.14</param>
+      </command_interface>
+      <state_interface name="position"/>
+    </joint>
+    <joint name="front_left_thigh_joint">
+      <command_interface name="position">
+        <param name="min">-3.14</param>
+        <param name="max">3.14</param>
+      </command_interface>
+      <state_interface name="position"/>
+    </joint>
+    <joint name="front_right_thigh_joint">
+      <command_interface name="position">
+        <param name="min">-3.14</param>
+        <param name="max">3.14</param>
+      </command_interface>
+      <state_interface name="position"/>
+    </joint>
+    <joint name="rear_left_thigh_joint">
+      <command_interface name="position">
+        <param name="min">-3.14</param>
+        <param name="max">3.14</param>
+      </command_interface>
+      <state_interface name="position"/>
+    </joint>
+    <joint name="rear_right_thigh_joint">
+      <command_interface name="position">
+        <param name="min">-3.14</param>
+        <param name="max">3.14</param>
+      </command_interface>
+      <state_interface name="position"/>
+    </joint>
+    <joint name="front_left_shin_joint">
+      <command_interface name="position">
+        <param name="min">-3.14</param>
+        <param name="max">3.14</param>
+      </command_interface>
+      <state_interface name="position"/>
+    </joint>
+    <joint name="front_right_shin_joint">
+      <command_interface name="position">
+        <param name="min">-3.14</param>
+        <param name="max">3.14</param>
+      </command_interface>
+      <state_interface name="position"/>
+    </joint>
+    <joint name="rear_left_shin_joint">
+      <command_interface name="position">
+        <param name="min">-3.14</param>
+        <param name="max">3.14</param>
+      </command_interface>
+      <state_interface name="position"/>
+    </joint>
+    <joint name="rear_right_shin_joint">
+      <command_interface name="position">
+        <param name="min">-3.14</param>
+        <param name="max">3.14</param>
+      </command_interface>
+      <state_interface name="position"/>
+    </joint>
+  </ros2_control>
+  <gazebo>
+    <plugin
+        filename="gz_ros2_control-system"
+        name="gz_ros2_control::GazeboSimROS2ControlPlugin">
+        <parameters>$(find robot)/config/robot_controller.yaml</parameters>
+    </plugin>
+    <plugin
+        filename="libgz-sim-joint-state-publisher-system"
+        name="gz::sim::systems::JointStatePublisher">
+    </plugin>
+    <plugin
+        filename="libgz-sim-pose-publisher-system"
+        name="gz::sim::systems::PosePublisher">
+        <publish_link_pose>true</publish_link_pose>
+        <use_pose_vector_msg>true</use_pose_vector_msg>
+        <publish_nested_model_pose>true</publish_nested_model_pose>
+    </plugin>
+    <plugin
+        filename="ignition-gazebo-sensors-system"
+        name="ignition::gazebo::systems::Sensors">
+        <render_engine>ogre2</render_engine>
+    </plugin>
+    <plugin
+        filename="gz-sim-imu-system"
+        name="gz::sim::systems::Imu">
+    </plugin>
+  </gazebo>
+</xacro:macro >
 </robot>
