Commit message: add environment

File: colcon_ws/src/robot/urdf/parts/base/base.xacro (robot description, xacro)
@@ -11,10 +11,12 @@
 	  <visual>
 		  <geometry>
-		    <mesh filename="package://robot/meshes/DAE/base/base_link.dae"/>
+		    <mesh filename="/home/alex/Documentos/universidad/robot/colcon_ws/src/robot/meshes/base_link.dae"
+        scale="1 1 1"/>
 		  </geometry>
 	  </visual>
 	  <collision>
 		  <geometry>
-		    <mesh filename="package://robot/meshes/STL/base/base_link.stl"/>
+		    <mesh filename="/home/alex/Documentos/universidad/robot/colcon_ws/src/robot/meshes/base_link.stl"
+        scale="1 1 1"/>
 		  </geometry>
 	  </collision>

File: colcon_ws/src/robot/urdf/parts/left_thigh/left_thigh.xacro (robot description, xacro)
@@ -14,10 +14,10 @@
 	  <visual>
 		<geometry>
-		  <mesh filename="package://robot/meshes/DAE/left_thigh/left_thigh.dae"/>
+		  <mesh filename="/home/alex/Documentos/universidad/robot/colcon_ws/src/robot/meshes/left_thigh.dae"/>
 		</geometry>
 	  </visual>
 	  <collision>
 		<geometry>
-		  <mesh filename="package://robot/meshes/STL/left_thigh/left_thigh.stl"/>
+		  <mesh filename="/home/alex/Documentos/universidad/robot/colcon_ws/src/robot/meshes/left_thigh.stl"/>
 		</geometry>
 	  </collision>

File: colcon_ws/src/robot/urdf/parts/leg_joint/leg_joint.xacro (robot description, xacro)
@@ -14,10 +14,10 @@
 	  <visual>
 		<geometry>
-		  <mesh filename="package://meshes/DAE/leg_joint/leg_joint.dae"/>
+		  <mesh filename="/home/alex/Documentos/universidad/robot/colcon_ws/src/robot/meshes/leg_joint.dae"/>
 		</geometry>
 	  </visual>
 	  <collision>
 		<geometry>
-		  <mesh filename="package://meshes/STL/leg_joint/leg_joint.stl"/>
+		  <mesh filename="/home/alex/Documentos/universidad/robot/colcon_ws/src/robot/meshes/leg_joint.stl"/>
 		</geometry>
 	  </collision>

File: colcon_ws/src/robot/urdf/parts/right_thigh/right_thigh.xacro (robot description, xacro)
@@ -14,10 +14,10 @@
 	  <visual>
 		<geometry>
-		  <mesh filename="package://robot/meshes/DAE/right_thigh/right_thigh.dae"/>
+		  <mesh filename="/home/alex/Documentos/universidad/robot/colcon_ws/src/robot/meshes/right_thigh.dae"/>
 		</geometry>
 	  </visual>
 	  <collision>
 		<geometry>
-		  <mesh filename="package://robot/meshes/STL/right_thigh/right_thigh.stl"/>
+		  <mesh filename="/home/alex/Documentos/universidad/robot/colcon_ws/src/robot/meshes/right_thigh.stl"/>
 		</geometry>
 	  </collision>

File: colcon_ws/src/robot/urdf/parts/shin/shin.xacro (robot description, xacro)
@@ -14,10 +14,10 @@
 	  <visual>
 		<geometry>
-		  <mesh filename="package://robot/meshes/DAE/shin/shin.dae"/>
+		  <mesh filename="/home/alex/Documentos/universidad/robot/colcon_ws/src/robot/meshes/shin.dae"/>
 		</geometry>
 	  </visual>
 	  <collision>
 		<geometry>
-		  <mesh filename="package://robot/meshes/STL/shin/shin.stl"/>
+		  <mesh filename="/home/alex/Documentos/universidad/robot/colcon_ws/src/robot/meshes/shin.stl"/>
 		</geometry>
 	  </collision>

File: colcon_ws/src/robot/urdf/robot.xacro (robot description, xacro)
@@ -65,4 +65,5 @@
   <!-- Controllers -->
   <!-- Base -->
+  <xacro:robot_ros2_control/>
   <!-- Base -->
   <xacro:base_gazebo_v0/>

Commit message: conflicts with collisions are solved

File: colcon_ws/src/robot/urdf/parts/base/base.xacro (robot description, xacro)
@@ -31,6 +31,6 @@
                 <mu>0.8</mu>
                 <mu2>0.8</mu2>
-                <kp>1e15</kp>
-                <kd>1e13</kd>
+                <kp>1000.0</kp>
+                <kd>0.1</kd>
               </ode>
             </friction>

File: colcon_ws/src/robot/urdf/parts/left_thigh/left_thigh.xacro (robot description, xacro)
@@ -25,5 +25,5 @@
 		<origin xyz="0.17 -0.028 0.014"/>
 		<mass value="1.24"/>
-		<inertia ixx="0.002" ixy="0" ixz="0" iyy="0.002" iyz="0" izz="0.001" />
+		<inertia ixx="0.002" ixy="0.0" ixz="0.0" iyy="0.002" iyz="0.0" izz="0.001" />
 		<!-- inertia ixx="-0.5" ixy="0.003" ixz="0.145" iyy="-0.496" iyz="-0.0096" izz="0.012" -->
 	  </inertial>

File: colcon_ws/src/robot/urdf/parts/leg_joint/leg_joint.xacro (robot description, xacro)
@@ -7,5 +7,5 @@
 	  <parent link="${parent}"/>
 	  <child link="${prefix}_leg_joint_link"/>
-          <limit effort="500" velocity="10" lower="-3.14159" upper = "3.14159"/>
+			<limit effort="500" velocity="10" lower="-3" upper = "3"/>
           <dynamics damping="0.005" friction="0.1"/>
 	  <xacro:insert_block name="joint_axis"/>

File: colcon_ws/src/robot/urdf/parts/right_thigh/right_thigh.xacro (robot description, xacro)
@@ -7,6 +7,6 @@
 	  <parent link="${parent}"/>
 	  <child link="${prefix}_right_thigh_link"/>
-          <limit effort="500" velocity="10" lower="-3" upper = "3"/>
-          <dynamics damping="0.005" friction="0.1"/>
+			<limit effort="500" velocity="10" lower="-3" upper = "3"/>
+        <dynamics damping="0.005" friction="0.1"/>
 	  <xacro:insert_block name="joint_axis"/>
 	</joint>

File: colcon_ws/src/robot/urdf/parts/shin/shin.xacro (robot description, xacro)
@@ -7,6 +7,6 @@
 	  <parent link="${parent}"/>
 	  <child link="${prefix}_shin_link"/>
-          <limit effort="500" velocity="10" lower="-3.14159" upper = "3.14159"/>
-          <dynamics damping="0.005" friction="0.1"/>
+		<limit effort="500" velocity="10" lower="-3" upper = "3"/>
+       <dynamics damping="0.005" friction="0.1"/>
 	  <xacro:insert_block name="joint_axis"/>
 	</joint>
@@ -18,4 +18,5 @@
 	  </visual>
 	  <collision>
+	  	<origin xyz="0 0 0" rpy="1.570796 0 0"/>
 		<geometry>
 		  <mesh filename="/home/alex/Documentos/universidad/robot/colcon_ws/src/robot/meshes/shin.stl"/>

Commit message: initilize robot

File: colcon_ws/src/robot/urdf/parts/base/base.xacro (robot description, xacro)
@@ -16,7 +16,11 @@
 	  </visual>
 	  <collision>
+      <!--<origin
+        xyz="0 0 0.07"
+        rpy="0 0 0" /> -->
 		  <geometry>
 		    <mesh filename="/home/alex/Documentos/universidad/robot/colcon_ws/src/robot/meshes/base_link.stl"
         scale="1 1 1"/>
+        <!--<box size="0.759 0.22 0.14"/>-->
 		  </geometry>
 	  </collision>
@@ -29,6 +33,6 @@
             <friction>
               <ode>
-                <mu>0.8</mu>
-                <mu2>0.8</mu2>
+                <mu>0.9</mu>
+                <mu2>0.9</mu2>
                 <kp>1e15</kp>
                 <kd>1e13</kd>

File: colcon_ws/src/robot/urdf/parts/left_thigh/left_thigh.xacro (robot description, xacro)
@@ -7,6 +7,6 @@
 	  <parent link="${parent}"/>
 	  <child link="${prefix}_left_thigh_link"/>
-          <limit effort="500" velocity="10" lower="-3" upper = "3"/>
-          <dynamics damping="0.005" friction="0.1"/>
+          <limit effort="0.001" velocity="10" lower="-3" upper = "3"/>
+          <dynamics damping="0.001" friction="0.7"/>
 	  <xacro:insert_block name="joint_axis"/>
 	</joint>
@@ -18,6 +18,10 @@
 	  </visual>
 	  <collision>
+	  <!--<origin
+        xyz="0.213 -0.03 0"
+        rpy="0 1.57075 0" /> -->
 		<geometry>
 		  <mesh filename="/home/alex/Documentos/universidad/robot/colcon_ws/src/robot/meshes/left_thigh.stl"/>
+		   <!-- <cylinder length="0.426" radius="0.035"/> -->
 		</geometry>
 	  </collision>

File: colcon_ws/src/robot/urdf/parts/leg_joint/leg_joint.xacro (robot description, xacro)
@@ -7,6 +7,6 @@
 	  <parent link="${parent}"/>
 	  <child link="${prefix}_leg_joint_link"/>
-			<limit effort="500" velocity="10" lower="-3" upper = "3"/>
-          <dynamics damping="0.005" friction="0.1"/>
+			<limit effort="0.001" velocity="10" lower="-3" upper = "3"/>
+          <dynamics damping="0.001" friction="0.1"/>
 	  <xacro:insert_block name="joint_axis"/>
 	</joint>

File: colcon_ws/src/robot/urdf/parts/right_thigh/right_thigh.xacro (robot description, xacro)
@@ -7,6 +7,6 @@
 	  <parent link="${parent}"/>
 	  <child link="${prefix}_right_thigh_link"/>
-			<limit effort="500" velocity="10" lower="-3" upper = "3"/>
-        <dynamics damping="0.005" friction="0.1"/>
+			<limit effort="0.001" velocity="10" lower="-3" upper = "3"/>
+        <dynamics damping="0.001" friction="0.7"/>
 	  <xacro:insert_block name="joint_axis"/>
 	</joint>
@@ -18,6 +18,11 @@
 	  </visual>
 	  <collision>
+	  <!--<origin
+			xyz="0.213 -0.03 0"
+			rpy="0 1.57075 0" />-->
 		<geometry>
 		  <mesh filename="/home/alex/Documentos/universidad/robot/colcon_ws/src/robot/meshes/right_thigh.stl"/>
+			<!--<mesh filename="/home/alex/Documentos/universidad/robot/colcon_ws/src/robot/meshes/left_thigh.stl"/>-->
+			<!--<cylinder length="0.426" radius="0.035"/>-->
 		</geometry>
 	  </collision>

File: colcon_ws/src/robot/urdf/parts/shin/shin.xacro (robot description, xacro)
@@ -8,5 +8,5 @@
 	  <child link="${prefix}_shin_link"/>
 		<limit effort="500" velocity="10" lower="-3" upper = "3"/>
-       <dynamics damping="0.005" friction="0.1"/>
+       <dynamics damping="0.01" friction="100"/>
 	  <xacro:insert_block name="joint_axis"/>
 	</joint>
@@ -18,7 +18,11 @@
 	  </visual>
 	  <collision>
-	  	<origin xyz="0 0 0" rpy="1.570796 0 0"/>
+	  		 <!-- <origin
+			xyz="-0.1825 0.012 0"
+			rpy="0 1.57075 0" /> -->
+			<origin xyz="0 0 0" rpy="1.570796 0 0"/>
 		<geometry>
 		  <mesh filename="/home/alex/Documentos/universidad/robot/colcon_ws/src/robot/meshes/shin.stl"/>
+		  <!--<cylinder length="0.345" radius="0.025"/>-->
 		</geometry>
 	  </collision>

File: colcon_ws/src/robot/urdf/robot_control_gazebo.xacro (robot description, xacro)
@@ -12,4 +12,5 @@
       </command_interface>
       <state_interface name="position"/>
+      <!--<state_interface name="velocity"/>-->
     </joint>
     <joint name="front_right_leg_joint">
@@ -19,4 +20,5 @@
       </command_interface>
       <state_interface name="position"/>
+     <!--<state_interface name="velocity"/>-->
     </joint>
     <joint name="rear_left_leg_joint">
@@ -26,4 +28,5 @@
       </command_interface>
       <state_interface name="position"/>
+      <!--<state_interface name="velocity"/>-->
     </joint>
     <joint name="rear_right_leg_joint">
@@ -33,4 +36,5 @@
       </command_interface>
       <state_interface name="position"/>
+ <!--<state_interface name="velocity"/>-->
     </joint>
     <joint name="front_left_thigh_joint">
@@ -40,4 +44,5 @@
       </command_interface>
       <state_interface name="position"/>
+    <!--<state_interface name="velocity"/>-->
     </joint>
     <joint name="front_right_thigh_joint">
@@ -47,4 +52,5 @@
       </command_interface>
       <state_interface name="position"/>
+   <!--<state_interface name="velocity"/>-->
     </joint>
     <joint name="rear_left_thigh_joint">
@@ -54,4 +60,5 @@
       </command_interface>
       <state_interface name="position"/>
+  <!--<state_interface name="velocity"/>-->
     </joint>
     <joint name="rear_right_thigh_joint">
@@ -61,4 +68,5 @@
       </command_interface>
       <state_interface name="position"/>
+   <!--<state_interface name="velocity"/>-->
     </joint>
     <joint name="front_left_shin_joint">
@@ -68,4 +76,5 @@
       </command_interface>
       <state_interface name="position"/>
+    <!--<state_interface name="velocity"/>-->
     </joint>
     <joint name="front_right_shin_joint">
@@ -75,4 +84,5 @@
       </command_interface>
       <state_interface name="position"/>
+  <!--<state_interface name="velocity"/>-->
     </joint>
     <joint name="rear_left_shin_joint">
@@ -82,4 +92,5 @@
       </command_interface>
       <state_interface name="position"/>
+<!--<state_interface name="velocity"/>-->
     </joint>
     <joint name="rear_right_shin_joint">
@@ -89,9 +100,10 @@
       </command_interface>
       <state_interface name="position"/>
+<!--<state_interface name="velocity"/>-->
     </joint>
   </ros2_control>
   <gazebo>
     <plugin filename="libgazebo_ros2_control.so" name="gazebo_ros2_control">
-        <parameters>$(find robot)/config/robot_controller.yaml</parameters>
+        <parameters>$(find robot)/config/robot_controller_forward.yaml</parameters>
          <controller_manager_node_name>controller_manager</controller_manager_node_name>
     </plugin>
